File: Prototoype 2 RevC/Tiles_Proto2.brd (EAGLE design)
At the start: 43.2 x 46.4 mm, 43 parts, among them J1 7p-SMD-2.54, Q1 MMBT3904LT1G, U1 ADXL345BCCZ-RL, U2 MPR121QR2, U3 MCP73832T-2ACI/OT-SOT23-5, U4 AT42QT1070-SSU

Commit message: refactoring
Parts:
- removed BOTTOM, LEFT, RIGHT, TOP: (no value), wirepad:SMD2,54-5,08
- removed C2, C3: 100NF 10V, Seeed-OPL-Capacitor:C0402
- removed CP7, CP8: (no value), wirepad:SMD1,27-2,54
- removed JP3: (no value), SparkFun-Connectors:1X08_ROUND
- removed R4: 75K 1/10W, Seeed-OPL-Resistor:R0603
- removed R7: 10K, Seeed-OPL-Resistor:R0603
- removed SJ1: JUMPER-PAD-2-NC_BY_TRACE, SparkFun-Passives:PAD-JUMPER-2-NC_BY_TRACE_YES_SILK
- removed U2: MPR121QR2, Seeed-OPL-sensor:QFN20-0.4-3X3M
- removed U4: AT42QT1070-SSU, Seeed-OPL-sensor:SOIC14-1.27-9.3X4.3MM
- moved B+ 1.27 mm to (24.1, 54.0)
- moved B- 1.27 mm to (27.3, 54.0)
- moved M+ 1.27 mm to (31.1, 54.0)
- moved M- 1.27 mm to (34.3, 54.0)
Connections:
- removed net N$16: LEFT.1, U2.8
- removed net N$17: RIGHT.1, U2.9
- removed net N$18: TOP.1, U2.10
- removed net N$19: BOTTOM.1, U2.11
- removed net N$20: CP7.1, U2.15
- removed net N$21: CP8.1, U2.16
- removed net N$24: C2.2, R7.2, SJ1.2, U2.20
- removed net N$4: C3.2, U2.5
- removed net N$5: R4.2, U2.7
- net GND: no longer C2.1, C3.1, R4.1, U2.4, U2.6
- net INT: now also U1.8; no longer R7.1, U2.1
- net SCL: no longer U2.2
- net SDA: no longer U2.3
- net VCC: no longer SJ1.1
Routing:
- net N$16: track 56.7 -> 0.00 mm, vias 1 -> 0
- net N$19: track 49.5 -> 0.00 mm, vias 1 -> 0
- net N$18: track 33.5 -> 0.00 mm, vias 1 -> 0
- net SDA: track 78.8 -> 50.2 mm
- net GND: track 167.0 -> 144.3 mm, vias 10 -> 8
- net N$24: track 22.3 -> 0.00 mm, vias 2 -> 0
- net N$5: track 9.24 -> 0.00 mm, vias 2 -> 0
- net N$17: track 8.82 -> 0.00 mm, vias 1 -> 0
- net N$20: track 5.65 -> 0.00 mm
- net N$21: track 5.28 -> 0.00 mm
- net SCL: track 45.5 -> 40.7 mm
- net INT: track 47.7 -> 51.4 mm, vias 4 -> 2
- net N$4: track 2.65 -> 0.00 mm
- net VCC: track 111.4 -> 109.4 mm
Other:
- board text added: "P#2 RevC (2016)"
- board text removed: "P#2 RevB (2016)"
- board text removed: "TOUCH PORTS"
