File: Prototoype 2 RevC/Tiles_Proto2.sch (EAGLE design)
At the start: 43 parts, among them J1 7p-SMD-2.54, Q1 MMBT3904LT1G, U1 ADXL345BCCZ-RL, U2 MPR121QR2, U3 MCP73832T-2ACI/OT-SOT23-5, U4 AT42QT1070-SSU

Commit message: refactoring
Parts:
- removed BOTTOM, LEFT, RIGHT, TOP: (no value), wirepad:SMD5
- removed C2, C3: 100NF 10V, Seeed-OPL-Capacitor:CERAMIC 100NF-10V-10%-X5R(0402)
- removed CP7, CP8: (no value), wirepad:SMD2
- removed JP3: (no value), SparkFun-Connectors:M08
- removed R4: 75K 1/10W, Seeed-OPL-Resistor:SMD-RES-75K-1%-1/10W(0603)
- removed R7: 10K, Seeed-OPL-Resistor:SMD-RES-10K-1%-1/10W(0603)
- removed SJ1: JUMPER-PAD-2-NC_BY_TRACE, SparkFun-Passives:JUMPER-PAD-2-NC_BY_TRACE
- removed U2: MPR121QR2, Seeed-OPL-sensor:TOUCH-MPR121QR2(QFN20)
- removed U4: AT42QT1070-SSU, Seeed-OPL-sensor:TOUCH-AT42QT1070-SSU(SOIC14)
Connections:
- removed net N$16: LEFT.P, U2.ELE0
- removed net N$17: RIGHT.P, U2.ELE1
- removed net N$18: TOP.P, U2.ELE2
- removed net N$19: BOTTOM.P, U2.ELE3
- removed net N$20: CP7.P, U2.ELE7
- removed net N$21: CP8.P, U2.ELE8
- removed net N$24: C2.2, R7.2, SJ1.2, U2.VDD
- removed net N$4: C3.2, U2.VREG
- removed net N$5: R4.2, U2.REXT
- net GND: no longer C2.1, C3.1, R4.1, U2.ADDR, U2.VSS
- net INT: now also U1.INT1; no longer R7.1, U2.!IRQ
- net SCL: no longer U2.SCL
- net SDA: no longer U2.SDA
- net VCC: no longer SJ1.1
Other:
- moved on the sheet: JP2
