File: Dock/Dock P1RA.sch (EAGLE design)
At the start: 14 parts, among them J2 MF-CON-2.54mm-01x07, J3 MF-CON-2.54mm-01x05, U1 MCP73831T-2ACI/OT

Commit message: switched imu from LSM9DS1 to ADXL345
Parts:
- C1, C2: device microbuilder:CAP_CERAMIC0805 -> microbuilder:CAP_CERAMIC1206
Changed lines of the file:
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@@
 <part name="R2" library="microbuilder" deviceset="RESISTOR" device="0805" value="470"/>
 <part name="U$2" library="microbuilder" deviceset="GND" device=""/>
-<part name="C1" library="microbuilder" deviceset="CAP_CERAMIC" device="0805" value="10µF"/>
+<part name="C1" library="microbuilder" deviceset="CAP_CERAMIC" device="1206" value="10µF"/>
 <part name="U$3" library="microbuilder" deviceset="GND" device=""/>
-<part name="C2" library="microbuilder" deviceset="CAP_CERAMIC" device="0805" value="10µF"/>
+<part name="C2" library="microbuilder" deviceset="CAP_CERAMIC" device="1206" value="10µF"/>
 <part name="U$5" library="microbuilder" deviceset="GND" device=""/>
 <part name="R3" library="microbuilder" deviceset="RESISTOR" device="0805" value="10K\"/>
