File: Prototype 3 RevA/Tiles_Proto3_RevA.sch (EAGLE design)
At the start: 40 parts, among them U2 MF-DSC-SOT233-MMBT3904

Commit message: p3rA and dock p1rA sent to production
Parts:
- removed C3: 10uf, Seeed-OPL-Capacitor:CERAMIC-10UF-10V-10%-X5R(0603)
- removed C4: 220nf, Seeed-OPL-Capacitor:CERAMIC-220NF-25V-10%-X7R(0603)
- IMU: value LSM9DS1 -> ADXL345BCCZ-RL; device LSM9DS1:LSM9DS1 -> Seeed-OPL-sensor:MOTION/POSITION-ADXL345BCCZ-RL(14P-5.0X3.0MM)
Connections:
- removed net N$1: C3.1, IMU.CAP
- removed net N$10: IMU.INT_M
- removed net N$12: IMU.INT2_A/G
- removed net N$2: C4.1, IMU.C1
- net GND: now also IMU.GND@1, IMU.GND@2, IMU.GND@3; no longer C3.2, C4.2, IMU.GND, IMU.RESERVED(GND)
- net IMU-INT: now also IMU.INT1; no longer IMU.INT1_A/G
- net SCL: now also IMU.SCL/SCLK; no longer IMU.SCL/SPC
- net SDA: now also IMU.SDA/SDI/SDIO; no longer IMU.SDA/SDI/SDO
- net VCC: now also IMU.!CS, IMU.VDDI/O, IMU.VS; no longer IMU.CS_A/G, IMU.CS_M, IMU.DEN_A/G, IMU.VDD, IMU.VDDIO
Other:
- moved on the sheet: C2
