File: Prototoype 2 RevD/Tiles_Proto2_RevD.sch (EAGLE design)
At the start: 30 parts, among them J1 4P-2.0-90D, J2 MF-CON-2.54mm-01x07, Q1 MMBT3904LT1G, U1 ADXL345BCCZ-RL, U3 MCP73832T-2ACI/OT-SOT23-5

Commit message: added proto 3 Rev B
Parts:
- R4: value (none) -> 27
- R5, R6: value (none) -> 22
Changed lines of the file:
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@@
 <?xml version="1.0" encoding="utf-8"?>
 <!DOCTYPE eagle SYSTEM "eagle.dtd">
-<eagle version="7.7.0">
+<eagle version="8.4.1">
 <drawing>
 <settings>
 <setting alwaysvectorfont="no"/>
+<setting keepoldvectorfont="yes"/>
 <setting verticaltext="up"/>
 </settings>
-<grid distance="0.1" unitdist="inch" unit="inch" style="lines" multiple="1" display="yes" altdistance="0.01" altunitdist="inch" altunit="inch"/>
+<grid distance="0.1" unitdist="inch" unit="inch" style="lines" multiple="1" display="no" altdistance="0.01" altunitdist="inch" altunit="inch"/>
 <layers>
 <layer number="1" name="Top" color="4" fill="1" visible="no" active="no"/>
@@
 <part name="J2" library="MF_Connectors" deviceset="CON_01X07" device="_PTH_2.54MM" value="MF-CON-2.54mm-01x07"/>
 <part name="D3" library="MF_LEDs" deviceset="LED_RGB_CA" device="_PLCC4" value="MF-LED-3228-RGB"/>
-<part name="R4" library="MF_Passives" deviceset="RESISTOR" device="_0603">
+<part name="R4" library="MF_Passives" deviceset="RESISTOR" device="_0603" value="27">
 <attribute name="HOUSEPART" value="MF-RES-0603-27"/>
 </part>
-<part name="R5" library="MF_Passives" deviceset="RESISTOR" device="_0603">
+<part name="R5" library="MF_Passives" deviceset="RESISTOR" device="_0603" value="22">
 <attribute name="HOUSEPART" value="MF-RES-0603-22"/>
 </part>
-<part name="R6" library="MF_Passives" deviceset="RESISTOR" device="_0603">
+<part name="R6" library="MF_Passives" deviceset="RESISTOR" device="_0603" value="22">
 <attribute name="HOUSEPART" value="MF-RES-0603-22"/>
 </part>
