File: Prototype 3 RevB/Tiles_Proto3_RevB.brd (EAGLE design)
At the start: 40 x 40 mm, 62 parts, among them Q1 DMG3415U-7, U2 MF-DSC-SOT233-MMBT3904, X1 32.768

Commit message: finished placing proto3revB
Parts:
- removed C12: 0.1uF, microbuilder2:0603-NO
- removed STAT1: MF-LED-0603-RED, MF_LEDs:LED0603
- added BTL: MF-LED-0603-RED, MF_LEDs:LED0603
- added C8: (no value), MF_Passives:C0603
- B+, B-: device wirepad:1,6/0,8 -> wirepad:SMD1,27-2,54
- C1: value 1uF -> (none)
- C10: value 10µF -> (none); device microbuilder2:0805-NO -> MF_Passives:C0805
- C11: value 10µF -> (none); device microbuilder2:0805-NO -> MF_Passives:C0603
- C2: value 100nf -> (none); device Seeed-OPL-Capacitor:C0603 -> MF_Passives:C0603
- C3: value 10uF -> (none)
- C4: value 22pF -> (none)
- C5: value 10uf -> (none); device Seeed-OPL-Capacitor:C0603 -> MF_Passives:C0603
- C6, C7: value 1uf -> (none); device Seeed-OPL-Capacitor:C0603 -> MF_Passives:C0603
- C9: value 22pF -> (none); device MF_Passives:C0603 -> MF_Passives:C0805
- J1: device tiles:1X07_SQUAREPADS_BOTTOM -> SparkFun-Connectors:1X07
- R1, R2, R3, R4, R7: value 10K 1/10W -> (none); device Seeed-OPL-Resistor:R0603 -> MF_Passives:R0603
- R10, R9: value 100K -> (none); device microbuilder2:0603-NO -> MF_Passives:R0603
- R11: value 10K -> (none); device microbuilder2:0603-NO -> MF_Passives:R0603
- R12, R13, R14, R15, R6: value 330 -> (none)
- R5: value 100K 1/10W -> (none); device Seeed-OPL-Resistor:R0603 -> MF_Passives:R0603
- R8: value 1K 1/10W -> (none); device Seeed-OPL-Resistor:R0603 -> MF_Passives:R0603
- TP2, TP3, TP4, TP5, TP6: device microbuilder2:PAD-1.5X2.0 -> microbuilder2:TESTPOINT_ROUND_2MM
- moved R14 131.7 mm to (26.2, -21.2), turned to 90 degrees
- moved D2 131.5 mm to (26.8, -6.97), turned to 180 degrees
- moved R13 127.8 mm to (26.2, -25.4), turned to 90 degrees
- moved R11 127.1 mm to (22.7, -7.00), turned to 180 degrees
- moved D3 127.0 mm to (20.2, -21.3)
- moved R9 125.7 mm to (31.7, -3.40)
- moved R10 121.5 mm to (23.1, 2.40), turned to 180 degrees
- moved C10 120.5 mm to (26.7, 1.50), turned to 270 degrees
- moved R12 120.2 mm to (20.1, -26.2)
- moved R15 113.7 mm to (8.84, -35.6)
- moved D1 110.2 mm to (8.44, 1.09), turned to 270 degrees
- moved SW1 109.0 mm to (7.79, -3.95), turned to 180 degrees
- moved U3 108.8 mm to (18.7, 1.34), turned to 180 degrees
- moved Q1 105.5 mm to (12.6, 1.33), turned to 90 degrees
- moved SJ1 98.9 mm to (-6.29, -10.9), turned to 180 degrees
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Connections:
- net 3.3V: now also C2.P$1, C5.P$1, C7.P$1, C9.P$1, R1.P$1, R11.P$2, R2.P$1, R3.P$1, R8.P$1; no longer C10.1, C2.1, C5.1, C7.2, R1.1, R11.1, R2.2, R3.2, R8.2
- net BUZZER: now also R7.P$2; no longer R7.2
- net CAP-INT: now also R3.P$2; no longer R3.1
- net CAP-RES: now also R4.P$1; no longer R4.2
- net DTR: now also C11.P$1; no longer C12.1
- net GND: now also BTL.CATHODE, C10.P$2, C2.P$2, C5.P$2, C6.P$2, C7.P$2, C8.P$2, R4.P$2, R5.P$2, R7.P$1, R9.P$2; no longer C10.2, C11.2, C2.2, C5.2, C6.1, C7.1, R4.1, R5.1, R7.1, R9.2, STAT1.CATHODE
- net N$10: now also R10.P$2; no longer R10.2
- net N$12: now also C8.P$1; no longer C9.P$1
- net N$13: now also C10.P$1, R10.P$1; no longer C11.1, R10.1
- net N$18: now also BTL.ANODE; no longer STAT1.ANODE
- net N$20: now also C11.P$2; no longer C12.2
- net N$3: now also R5.P$1; no longer R5.2
- net N$4: now also R8.P$2; no longer R8.1
- net N$5: now also C6.P$1; no longer C6.2
- net RESET: now also R11.P$1; no longer R11.2
- net SCL: now also R1.P$2; no longer R1.2
- net SDA: now also R2.P$2; no longer R2.1
- net VBUS: now also R9.P$1; no longer R9.1
Routing:
- net GND: track 120.2 -> 0.00 mm, vias 12 -> 0
- net SDA: track 73.7 -> 0.00 mm, vias 3 -> 0
- net SCL: track 72.4 -> 0.00 mm, vias 6 -> 0
- net IO-3: track 50.7 -> 0.00 mm, vias 2 -> 0
- net 3.3V: track 47.9 -> 0.00 mm
- net N$8: track 42.1 -> 0.00 mm, vias 1 -> 0
- net BUZZER: track 41.4 -> 0.00 mm, vias 2 -> 0
- net IO-2: track 37.5 -> 0.00 mm, vias 1 -> 0
- net N$7: track 33.4 -> 0.00 mm, vias 2 -> 0
- net CAP-A: track 27.4 -> 0.00 mm, vias 1 -> 0
- net CAP-B: track 25.2 -> 0.00 mm, vias 1 -> 0
- net IMU-INT: track 23.7 -> 0.00 mm, vias 2 -> 0
- net CAP-INT: track 22.1 -> 0.00 mm, vias 2 -> 0
- net CAP-RES: track 21.0 -> 0.00 mm, vias 2 -> 0
- net BTN: track 18.2 -> 0.00 mm, vias 2 -> 0
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- removed copper zone on layer 1, net GND
- removed copper zone on layer 16, net GND
Other:
- board outline removed
- board text removed: "/Users/Simone/Downloads/digi.bmp"
- board text removed: "00"
- board text removed: "01"
- board text removed: "BAT"
- board text removed: "FAC"
- board text removed: "RST"

Commit message: partial routing
Parts:
- removed TP1: (no value), microbuilder2:PAD-1.5X2.0
- removed TP2, TP3, TP4, TP5, TP6: (no value), microbuilder2:TESTPOINT_ROUND_2MM
- added DFU, RST, SWCLK, SWDIO, SWO: (no value), microbuilder2:TESTPOINT_ROUND_2MM
- added FRST: (no value), microbuilder2:PAD-1.5X2.0
- moved B- 23.9 mm to (22.5, -5.34), flipped to the bottom, turned to 270 degrees
- moved B+ 21.0 mm to (15.4, -5.35), flipped to the bottom, turned to 270 degrees
- moved R2 14.1 mm to (27.4, -32.5), turned to 90 degrees
- moved SJ1 12.7 mm to (1.80, -20.8), flipped to the bottom, turned to 270 degrees
- moved R1 12.5 mm to (30.2, -32.5), turned to 90 degrees
- moved BUZZER 10.9 mm to (38.8, -28.5)
- moved C4 7.53 mm to (24.7, -9.91)
- moved C2 7.21 mm to (32.4, -32.5), turned to 270 degrees
- moved C8 6.20 mm to (24.8, -17.2)
- moved HAPTIC 3.31 mm to (31.0, -23.2)
- moved C6 3.31 mm to (29.8, -19.7)
- moved C7 3.31 mm to (33.8, -19.7)
- moved IMU 3.28 mm to (31.1, -28.1)
- moved TOUCH 1.80 mm to (-1.23, -20.2)
- moved X1 1.39 mm to (24.7, -13.0), turned to 90 degrees
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Connections:
- net DFU: now also DFU.P$1; no longer TP5.P$1
- net FRST: now also FRST.P$1; no longer TP1.P$1
- net RESET: now also RST.P$1; no longer TP4.P$1
- net SWCLK: now also SWCLK.P$1; no longer TP3.P$1
- net SWDIO: now also SWDIO.P$1; no longer TP2.P$1
- net SWO: now also SWO.P$1; no longer TP6.P$1
Routing:
- net 3.3V: track 0.00 -> 143.8 mm, vias 0 -> 4
- net SCL: track 0.00 -> 87.1 mm, vias 0 -> 2
- net SDA: track 0.00 -> 79.3 mm, vias 0 -> 4
- net BT_LED: track 0.00 -> 42.9 mm
- net RESET: track 0.00 -> 37.5 mm, vias 0 -> 1
- net CAP-INT: track 0.00 -> 35.7 mm, vias 0 -> 2
- net CAP-RES: track 0.00 -> 34.1 mm, vias 0 -> 2
- net SWO: track 0.00 -> 29.8 mm, vias 0 -> 1
- net BTN: track 0.00 -> 29.1 mm, vias 0 -> 2
- net DTR: track 0.00 -> 28.8 mm, vias 0 -> 1
- net STATLED: track 0.00 -> 27.7 mm, vias 0 -> 2
- net N$13: track 0.00 -> 27.3 mm
- net IMU-INT: track 0.00 -> 25.1 mm, vias 0 -> 2
- net LED_R: track 0.00 -> 21.8 mm, vias 0 -> 2
- net SWCLK: track 0.00 -> 21.7 mm, vias 0 -> 1
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- added copper zone on layer 1, net GND

Commit message: ready for prod
Parts:
- removed CAP: (no value), cap1188-microbuilder:QFN24_4MM_SMSC
- removed IMU: ADXL345BCCZ-RL, Seeed-OPL-sensor:LGA14-0.8-5.0X3.0MM
- added EN: (no value), SparkFun-Connectors:1X02_NO_SILK
- added T2: MF-DSC-SOT233-MMBT3904, MF_Discrete_Semiconductor:SOT-23-3
- added U4: CAP1188, cap1188-microbuilder:QFN24_4MM_SMSC
- U1: value (none) -> MDBT42Q
- U2: value MF-DSC-SOT233-MMBT3904 -> AP2112; device MF_Discrete_Semiconductor:SOT-23-3 -> microbuilder2:SOT23-5
- U3: value (none) -> ADXL345; device microbuilder2:SOT23-5 -> Seeed-OPL-sensor:LGA14-0.8-5.0X3.0MM
- moved U2 40.9 mm to (18.2, 1.34), turned to 180 degrees
- moved U3 32.1 mm to (31.1, -28.1), turned to 90 degrees
- moved C11 2.38 mm to (10.2, -23.6)
- moved C3 2.38 mm to (14.4, -23.6)
- moved C5 2.38 mm to (10.2, -27.2)
- moved R3 2.38 mm to (10.2, -30.7)
- moved R4 2.38 mm to (14.4, -27.2)
- moved R5 2.38 mm to (14.4, -30.7)
- moved C9 2.00 mm to (29.9, 1.37)
- moved SW 2.00 mm to (20.0, -29.4)
- moved B+ 1.47 mm to (16.7, -6.04)
- moved SWO 1.39 mm to (1.86, -18.3)
- moved RST 1.35 mm to (4.70, -21.7)
- moved GPIO 1.35 mm to (39.4, -15.8)
- moved L1 1.32 mm to (13.4, -20.7)
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- renumbered HAPTIC to U5
Connections:
- removed net N$10: R10.P$2, U3.3
- new net EN: EN.1, R10.P$2, U2.3
- net 3.3V: now also U2.5, U3.1, U3.6, U3.7, U4.23; no longer CAP.23, IMU.1, IMU.6, IMU.7, U3.5
- net BUZZER: now also T2.P$1; no longer U2.P$1
- net CAP-A: now also U4.22; no longer CAP.22
- net CAP-B: now also U4.21; no longer CAP.21
- net CAP-INT: now also U4.13; no longer CAP.13
- net CAP-RES: now also U4.24; no longer CAP.24
- net GND: now also EN.2, T2.P$2, U2.2, U3.4, U3.5, U4.1, U4.THERM; no longer CAP.1, CAP.THERM, IMU.2, IMU.4, IMU.5, U2.P$2
- net IMU-INT: now also U3.8; no longer IMU.8
- net N$13: now also U2.1; no longer U3.1
- net N$3: now also U4.14; no longer CAP.14
- net N$4: now also T2.P$3; no longer U2.P$3
- net SCL: now also U3.14, U4.4; no longer CAP.4, IMU.14
- net SDA: now also U3.13, U4.3; no longer CAP.3, IMU.13
Routing:
- net GND: track 2.52 -> 145.2 mm, vias 0 -> 11
- net BUZZER: track 4.95 -> 45.4 mm, vias 0 -> 2
- net CAP-A: track 0.00 -> 34.8 mm, vias 0 -> 1
- net CAP-B: track 0.00 -> 26.2 mm, vias 0 -> 1
- net EN: track 0.00 -> 21.2 mm, vias 0 -> 1
- net IO-3: track 21.2 -> 41.7 mm
- net N$7: track 0.00 -> 19.3 mm, vias 0 -> 1
- net 3.3V: track 143.8 -> 163.0 mm
- net IO-2: track 19.3 -> 37.0 mm
- net VBUS: track 13.1 -> 27.0 mm, vias 0 -> 1
- net RESET: track 37.5 -> 49.5 mm
- net VBAT: track 7.16 -> 13.8 mm
- net N$10: track 5.93 -> 0.00 mm
- net N$20: track 9.68 -> 12.2 mm
- net BT_LED: track 42.9 -> 41.2 mm
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- added copper zone on layer 16, net GND
Other:
- board outline added: 46 x 46 mm
- board text added: "3.3v"
- board text added: "DTR"
- board text added: "P#3 RevB (2017)"
- board text added: "RXD"
- board text added: "TXD"
- board text added: "VBAT"
- board text added: "VBU"
- board text added: "http://tilestoolkit.io"
- board text added: "simone.mora@ntnu.no"
- board text removed: "Make everyday things interactive http://tilestoolkit.io"
- board text removed: "P#3 RevA (2017)"
- board text removed: "Simone Mora"
- board text removed: "VCC"

Commit message: added dock p1rb
Parts:
- moved R9 5.83 mm to (34.7, -8.40)
- moved SWCLK 5.83 mm to (4.66, -18.4)
- moved B+ 5.83 mm to (19.7, -11.0)
- moved B- 5.83 mm to (24.4, -11.0)
- moved M- 5.83 mm to (41.3, -12.3)
- moved R11 5.83 mm to (26.0, -12.0)
- moved SW1 5.83 mm to (10.8, -9.33)
- moved BTL 5.83 mm to (11.9, -43.8)
- moved BUZZER 5.83 mm to (41.8, -33.5)
- moved C1 5.83 mm to (10.9, -25.7)
- moved C10 5.83 mm to (29.1, -3.75)
- moved C11 5.83 mm to (13.2, -28.6)
- moved C2 5.83 mm to (35.4, -37.5)
- moved C3 5.83 mm to (17.4, -28.6)
- moved C4 5.83 mm to (27.7, -14.9)
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Routing:
- net EN: track 21.2 -> 19.0 mm

Commit message: values back in sch
Parts:
- C1, C6, C7: value (none) -> 1uF
- C10, C5, C9: value (none) -> 10uF
- C11: value (none) -> 0.1uF
- C2: value (none) -> 100nF
- C4, C8: value (none) -> 22pF
- L1: value (none) -> 10uH
- R1, R11, R2, R3, R4, R7: value (none) -> 10K
- R10, R5, R9: value (none) -> 100K
- R12: value (none) -> 27
- R13, R14: value (none) -> 22
- R15, R6: value (none) -> 330
- R8: value (none) -> 1K

Commit message: re-added part values
Parts:
- C3: value (none) -> 10uF
Changed lines of the file:
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@@
 <attribute name="VOLTAGE" value="" x="10.923" y="-25.6815" size="1.778" layer="27" rot="R180" display="off"/>
 </element>
-<element name="C3" library="MF_Passives" package="C0603" value="" x="17.3749" y="-28.6458" smashed="yes" rot="R180">
+<element name="C3" library="MF_Passives" package="C0603" value="10uF" x="17.3749" y="-28.6458" smashed="yes" rot="R180">
 <attribute name="DIELECTRIC" value="" x="17.3749" y="-28.6458" size="1.778" layer="27" rot="R180" display="off"/>
 <attribute name="HOUSEPART" value="" x="17.3749" y="-28.6458" size="1.778" layer="27" rot="R180" display="off"/>

Commit message: ready for ready for prod
Routing:
- net GND: track 145.2 -> 145.8 mm
Changed lines of the file:
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@@
 <wire x1="15.954053125" y1="-26.844053125" x2="12.5181" y2="-26.844053125" width="0.254" layer="1"/>
 <via x="12.5181" y="-26.844053125" extent="1-16" drill="0.35"/>
-<wire x1="12.5181" y1="-26.844053125" x2="9.604053125" y2="-26.844053125" width="0.254" layer="16"/>
+<wire x1="9.604053125" y1="-26.844053125" x2="12.5181" y2="-26.844053125" width="0.254" layer="16"/>
 <wire x1="9.604053125" y1="-26.844053125" x2="9.604" y2="-26.844" width="0.254" layer="16"/>
-<via x="9.604" y="-26.844" extent="1-16" drill="0.35"/>
-<wire x1="9.604" y1="-26.844" x2="9.604" y2="-26.2505" width="0.254" layer="1"/>
-<wire x1="9.604" y1="-26.2505" x2="10.173" y2="-25.6815" width="0.254" layer="1"/>
 <wire x1="16.6249" y1="-27.5149" x2="15.954053125" y2="-26.844053125" width="0.254" layer="1"/>
-<wire x1="5.3114" y1="-29.5872" x2="5.3368" y2="-29.511" width="0.254" layer="1"/>
-<wire x1="6.9556" y1="-33.2678" x2="5.6096" y2="-31.9218" width="0.254" layer="1"/>
-<wire x1="5.6096" y1="-31.9218" x2="5.50139375" y2="-31.9218" width="0.254" layer="1"/>
-<wire x1="5.50139375" y1="-31.9218" x2="5.3114" y2="-31.73180625" width="0.254" layer="1"/>
-<wire x1="5.3114" y1="-31.73180625" x2="5.3114" y2="-29.5872" width="0.254" layer="1"/>
-<wire x1="6.01718125" y1="-28.13398125" x2="6.081359375" y2="-28.069803125" width="0.254" layer="1"/>
-<wire x1="6.081359375" y1="-28.069803125" x2="6.119765625" y2="-27.987575" width="0.254" layer="1"/>
-<wire x1="6.119765625" y1="-27.987575" x2="6.1885875" y2="-27.962575" width="0.254" layer="1"/>
-<wire x1="6.1885875" y1="-27.962575" x2="6.2403625" y2="-27.9108" width="0.254" layer="1"/>
-<wire x1="7.55123125" y1="-27.5298" x2="7.56196875" y2="-27.5190625" width="0.254" layer="1"/>
-<wire x1="7.56196875" y1="-27.5190625" x2="7.5771125" y2="-27.518015625" width="0.254" layer="1"/>
-<wire x1="7.5771125" y1="-27.518015625" x2="7.672078125" y2="-27.408953125" width="0.254" layer="1"/>
-<wire x1="7.672078125" y1="-27.408953125" x2="7.7744125" y2="-27.30661875" width="0.254" layer="1"/>
-<wire x1="5.3368" y1="-29.511" x2="5.54020625" y2="-29.15519375" width="0.254" layer="1"/>
-<wire x1="5.54020625" y1="-29.15519375" x2="6.01718125" y2="-28.13398125" width="0.254" layer="1"/>
-<wire x1="7.7744125" y1="-27.30661875" x2="8.1772375" y2="-26.844" width="0.254" layer="1"/>
-<wire x1="8.1772375" y1="-26.844" x2="9.604" y2="-26.844" width="0.254" layer="1"/>
-<wire x1="7.406909375" y1="-27.539771875" x2="7.55123125" y2="-27.5298" width="0.254" layer="1"/>
-<wire x1="6.2403625" y1="-27.9108" x2="7.261746875" y2="-27.539771875" width="0.254" layer="1"/>
-<wire x1="7.261746875" y1="-27.539771875" x2="7.406909375" y2="-27.539771875" width="0.254" layer="1"/>
 <wire x1="18.1249" y1="-32.2931" x2="18.1249" y2="-35.6858" width="0.254" layer="1"/>
 <wire x1="20.925" y1="-33.325" x2="19.891" y2="-34.359" width="0.254" layer="1"/>
@@
 <wire x1="15" y1="-45" x2="14.75" y2="-44.75" width="0.254" layer="1"/>
 <wire x1="14.75" y1="-44.75" x2="14.75" y2="-43.8" width="0.254" layer="1"/>
+<wire x1="4.9556" y1="-32.0178" x2="4.9556" y2="-30.0254" width="0.254" layer="1"/>
+<wire x1="4.9556" y1="-30.0254" x2="4.953" y2="-30.0228" width="0.254" layer="1"/>
+<wire x1="4.953" y1="-30.0228" x2="4.953" y2="-29.845" width="0.254" layer="1"/>
+<wire x1="4.953" y1="-29.845" x2="5.1562" y2="-29.6418" width="0.254" layer="1"/>
+<wire x1="5.1562" y1="-29.6418" x2="5.1562" y2="-29.2354" width="0.254" layer="1"/>
+<wire x1="5.1562" y1="-29.2354" x2="5.8706375" y2="-28.5209625" width="0.254" layer="1"/>
+<wire x1="5.8706375" y1="-28.5209625" x2="5.883103125" y2="-28.49426875" width="0.254" layer="1"/>
+<wire x1="5.883103125" y1="-28.49426875" x2="5.883103125" y2="-28.113215625" width="0.254" layer="1"/>
+<wire x1="5.883103125" y1="-28.113215625" x2="6.2738" y2="-27.559" width="0.254" layer="1"/>
+<wire x1="6.2738" y1="-27.559" x2="9.0932" y2="-27.559" width="0.254" layer="1"/>
+<wire x1="10.173" y1="-25.6815" x2="10.173" y2="-26.4792" width="0.254" layer="1"/>
+<wire x1="9.0932" y1="-27.559" x2="10.173" y2="-26.4792" width="0.254" layer="1"/>
+<wire x1="10.173" y1="-26.4792" x2="9.7288" y2="-26.035" width="0.254" layer="1"/>
+<wire x1="9.7288" y1="-26.035" x2="9.2964" y2="-26.035" width="0.254" layer="1"/>
+<via x="9.2964" y="-26.035" extent="1-16" drill="0.35"/>
+<wire x1="9.2964" y1="-26.035" x2="9.604053125" y2="-26.342653125" width="0.254" layer="16"/>
+<wire x1="9.604053125" y1="-26.342653125" x2="9.604053125" y2="-26.844053125" width="0.254" layer="16"/>
 </signal>
 <signal name="RESET">
@@
 <wire x1="21.2107875" y1="-22.3" x2="22.5797875" y2="-23.669" width="0.254" layer="1"/>
 <wire x1="22.5797875" y1="-23.669" x2="29.82781875" y2="-23.669" width="0.254" layer="1"/>
-<wire x1="30.051" y1="-23.44581875" x2="30.051" y2="-17.446" width="0.254" layer="1"/>
-<wire x1="30.051" y1="-17.446" x2="30.432" y2="-17.446" width="0.254" layer="1"/>
+<wire x1="30.051" y1="-23.44581875" x2="30.051" y2="-18.4112" width="0.254" layer="1"/>
 <wire x1="31.694" y1="-12.5052125" x2="31.694" y2="-11.4947875" width="0.254" layer="1"/>
 <wire x1="31.694" y1="-11.4947875" x2="31.5452125" y2="-11.346" width="0.254" layer="1"/>
@@
 <wire x1="31.5452125" y1="-11.346" x2="29.77439375" y2="-11.346" width="0.254" layer="1"/>
 <wire x1="29.77439375" y1="-11.346" x2="29.27889375" y2="-11.8415" width="0.254" layer="1"/>
-<wire x1="30.432" y1="-17.446" x2="30.432" y2="-13.7672125" width="0.254" layer="1"/>
-<wire x1="30.432" y1="-13.7672125" x2="31.694" y2="-12.5052125" width="0.254" layer="1"/>
+<wire x1="30.051" y1="-18.4112" x2="30.051" y2="-14.7324125" width="0.254" layer="1"/>
+<wire x1="30.051" y1="-14.7324125" x2="31.694" y2="-12.5052125" width="0.254" layer="1"/>
 </signal>
 <signal name="N$11">

Commit message: ready for prod
Parts:
- BTL: value MF-LED-0603-RED -> RED
- C10, C9: device MF_Passives:C0805 -> MF_Passives:C1206
- C2: value 100nF -> 0.1uF
- C3, C5: device MF_Passives:C0603 -> MF_Passives:C1206
- D2: device microbuilder2:SOD-323 -> MF_Discrete_Semiconductor:SOD-123
- D3: value MF-LED-3228-RGB -> RGBLED
- L1: device MF_Passives:L0603 -> MF_Passives:L1210
- STAT: value MF-LED-0603-RED -> WHITE
- SW: value MF-SW-TACT-4.2MM -> SW
- T2: value MF-DSC-SOT233-MMBT3904 -> MMBT3904
- moved M- 1.60 mm to (41.0, -10.7)
- moved D2 1.50 mm to (31.0, -12.1)
- moved R3 1.18 mm to (13.4, -36.9)
- moved R4 0.89 mm to (17.4, -33.1)
- moved R5 0.80 mm to (17.6, -36.4)
- moved C3 0.74 mm to (17.3, -29.4)
- moved C5 0.54 mm to (13.3, -32.7)
- moved L1 0.46 mm to (16.4, -26.1)
- moved FRST 0.41 mm to (4.19, -10.4)
- moved SWCLK 0.41 mm to (4.64, -18.8)
- moved C11 0.36 mm to (12.9, -28.6)
- moved C9 0.31 mm to (32.8, -3.93)
- moved C10 0.23 mm to (29.1, -3.98)
- moved SWDIO 0.18 mm to (4.70, -14.2)
- moved M+ 0.16 mm to (37.8, -9.77)
- renumbered SW1 to RESW
Connections:
- net 3.3V: now also D2.CATHODE; no longer D2.C
- net RESET: now also D2.ANODE; no longer D2.A
Routing:
- net 3.3V: track 162.6 -> 169.1 mm
- net RESET: track 49.5 -> 53.1 mm
- net CAP-INT: track 35.0 -> 37.8 mm
- net CAP-RES: track 35.2 -> 36.4 mm
- net N$7: track 19.3 -> 20.2 mm
- net N$20: track 12.2 -> 12.9 mm
