File: Dock P1RB/Dock P1RB.brd (EAGLE design)
At the start: 41 x 46 mm, 16 parts, among them U1 MCP73831T-2ACI/OT

Commit message: dock ready for prod
Parts:
- removed C: RED, microbuilder:CHIPLED_0805
- removed R: GREEN, microbuilder:CHIPLED_0805
- added D1: MF-LED-0805-RED, MF_LEDs:LED0805
- added D2: MF-LED-0805-GREEN, MF_LEDs:LED0805
- C1, C2, C4: device MF_Passives:C0805 -> MF_Passives:C1206
- moved J1 6.00 mm to (28.0, -31.0)
Connections:
- net GND: now also D2.CATHODE; no longer R.C
- net N$1: now also D1.CATHODE; no longer C.C
- net N$6: now also D2.ANODE; no longer R.A
- net VBUS: now also D1.ANODE; no longer C.A
Routing:
- net VBUS: track 76.2 -> 83.6 mm
- net TXD: track 17.7 -> 23.7 mm
- net DTR: track 19.8 -> 25.8 mm
- net VBAT: track 18.4 -> 23.5 mm
- net 3.3V: track 36.7 -> 41.8 mm
- net RXD: track 15.3 -> 20.3 mm
- net GND: track 76.6 -> 81.0 mm
- net N$3: track 4.94 -> 4.44 mm
Other:
- board size 41 x 46 mm -> 44 x 46 mm
- board text added: "Tiles IoT Dock"

Commit message: cleanup
Parts:
- U2: value (none) -> CP2104
Changed lines of the file:
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@@
 <element name="H1" library="tiles" package="2,5-PAD-SIM" value="MOUNT-PAD-ROUND2.5" x="25" y="-5"/>
 <element name="H2" library="tiles" package="2,5-PAD-SIM" value="MOUNT-PAD-ROUND2.5" x="25" y="-41"/>
-<element name="U2" library="microbuilder2" package="QFN24_4MM_SMSC" value="" x="7" y="-17"/>
+<element name="U2" library="microbuilder2" package="QFN24_4MM_SMSC" value="CP2104" x="7" y="-17">
+<attribute name="HOUSEPART" value="no" x="7" y="-17" size="1.778" layer="27" display="off"/>
+<attribute name="MPN" value="CP2104" x="7" y="-17" size="1.778" layer="27" display="off"/>
+<attribute name="POPULATE" value="1" x="7" y="-17" size="1.778" layer="27" display="off"/>
+</element>
 <element name="C3" library="MF_Passives" package="C0603" value="0.1uF" x="6" y="-11" rot="R90">
 <attribute name="DIELECTRIC" value="" x="6" y="-11" size="1.778" layer="27" rot="R90" display="off"/>
