File: Dock P1RB/Dock P1RB.sch (EAGLE design)
At the start: 16 parts, among them U1 MCP73831T-2ACI/OT

Commit message: dock ready for prod
Parts:
- removed C: RED, microbuilder:LED0805
- removed R: GREEN, microbuilder:LED0805
- added D1: MF-LED-0805-RED, MF_LEDs:LED_SINGLE-0805-RED
- added D2: MF-LED-0805-GREEN, MF_LEDs:LED_SINGLE-0805-GREEN
- C1, C2, C4: device MF_Passives:CAPACITOR_NP_0805 -> MF_Passives:CAPACITOR_NP_1206; HOUSEPART (none) -> YES; MPN (none) -> MF-CAP-1206-10uF
- C3: HOUSEPART (none) -> YES; MPN (none) -> MF-CAP-0603-0.1uF
- R1, R2: HOUSEPART (none) -> YES; MPN (none) -> MF-RES-0603-470
- R3: HOUSEPART (none) -> YES; MPN (none) -> MF-RES-0603-10K
- R4: HOUSEPART (none) -> YES; MPN (none) -> MF-RES-0603-1K
- U1: HOUSEPAR (none) -> no; MPN (none) -> MCP73831T-2ACI/OT; POPULATE (none) -> 1
Connections:
- net GND: now also D2.CATHODE; no longer R.C
- net N$1: now also D1.CATHODE; no longer C.C
- net N$6: now also D2.ANODE; no longer R.A
- net VBUS: now also D1.ANODE; no longer C.A
Changed lines of the file:
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@@
 </classes>
 <parts>
-<part name="U1" library="microbuilder" deviceset="MCP73831/2" device="" value="MCP73831T-2ACI/OT"/>
+<part name="U1" library="microbuilder" deviceset="MCP73831/2" device="" value="MCP73831T-2ACI/OT">
+<attribute name="HOUSEPAR" value="no"/>
+<attribute name="MPN" value="MCP73831T-2ACI/OT"/>
+<attribute name="POPULATE" value="1"/>
+</part>
 <part name="CN1" library="microbuilder" deviceset="USB_TYPEA" device="PCB"/>
-<part name="C" library="microbuilder" deviceset="LED" device="0805" value="RED"/>
-<part name="R" library="microbuilder" deviceset="LED" device="0805" value="GREEN"/>
 <part name="U$2" library="microbuilder" deviceset="GND" device=""/>
 <part name="U$3" library="microbuilder" deviceset="GND" device=""/>
@@
 <part name="U$12" library="microbuilder" deviceset="GND" device=""/>
 <part name="U$13" library="microbuilder" deviceset="GND" device=""/>
-<part name="C3" library="MF_Passives" deviceset="CAPACITOR_NP" device="_0603" value="0.1uF"/>
-<part name="C4" library="MF_Passives" deviceset="CAPACITOR_NP" device="_0805" value="10uF"/>
-<part name="R4" library="MF_Passives" deviceset="RESISTOR" device="_0603" value="1K"/>
+<part name="C3" library="MF_Passives" deviceset="CAPACITOR_NP" device="_0603" value="0.1uF">
+<attribute name="HOUSEPART" value="YES"/>
+<attribute name="MPN" value="MF-CAP-0603-0.1uF"/>
+</part>
+<part name="C4" library="MF_Passives" deviceset="CAPACITOR_NP" device="_1206" value="10uF">
+<attribute name="HOUSEPART" value="YES"/>
+<attribute name="MPN" value="MF-CAP-1206-10uF"/>
+</part>
+<part name="R4" library="MF_Passives" deviceset="RESISTOR" device="_0603" value="1K">
+<attribute name="HOUSEPART" value="YES"/>
+<attribute name="MPN" value="MF-RES-0603-1K"/>
+</part>
 <part name="U$14" library="microbuilder2" deviceset="VBUS" device=""/>
-<part name="R1" library="MF_Passives" deviceset="RESISTOR" device="_0603" value="470"/>
-<part name="R2" library="MF_Passives" deviceset="RESISTOR" device="_0603" value="470"/>
-<part name="R3" library="MF_Passives" deviceset="RESISTOR" device="_0603" value="10K"/>
-<part name="C1" library="MF_Passives" deviceset="CAPACITOR_NP" device="_0805" value="10uF"/>
-<part name="C2" library="MF_Passives" deviceset="CAPACITOR_NP" device="_0805" value="10uF"/>
+<part name="R1" library="MF_Passives" deviceset="RESISTOR" device="_0603" value="470">
+<attribute name="HOUSEPART" value="YES"/>
+<attribute name="MPN" value="MF-RES-0603-470"/>
+</part>
+<part name="R2" library="MF_Passives" deviceset="RESISTOR" device="_0603" value="470">
+<attribute name="HOUSEPART" value="YES"/>
+<attribute name="MPN" value="MF-RES-0603-470"/>
+</part>
+<part name="R3" library="MF_Passives" deviceset="RESISTOR" device="_0603" value="10K">
+<attribute name="HOUSEPART" value="YES"/>
+<attribute name="MPN" value="MF-RES-0603-10K"/>
+</part>
+<part name="C1" library="MF_Passives" deviceset="CAPACITOR_NP" device="_1206" value="10uF">
+<attribute name="HOUSEPART" value="YES"/>
+<attribute name="MPN" value="MF-CAP-1206-10uF"/>
+</part>
+<part name="C2" library="MF_Passives" deviceset="CAPACITOR_NP" device="_1206" value="10uF">
+<attribute name="HOUSEPART" value="YES"/>
+<attribute name="MPN" value="MF-CAP-1206-10uF"/>
+</part>
 <part name="J1" library="SparkFun-Connectors" deviceset="CONN_07" device=""/>
+<part name="D1" library="MF_LEDs" deviceset="LED_SINGLE" device="-0805-RED" value="MF-LED-0805-RED"/>
+<part name="D2" library="MF_LEDs" deviceset="LED_SINGLE" device="-0805-GREEN" value="MF-LED-0805-GREEN"/>
 </parts>
 <sheets>
@@
 </plain>
 <instances>
-<instance part="U1" gate="G$1" x="124.46" y="144.78"/>
+<instance part="U1" gate="G$1" x="124.46" y="144.78">
+<attribute name="HOUSEPAR" x="124.46" y="144.78" size="1.778" layer="96" display="off"/>
+<attribute name="MPN" x="124.46" y="144.78" size="1.778" layer="96" display="off"/>
+<attribute name="POPULATE" x="124.46" y="144.78" size="1.778" layer="96" display="off"/>
+</instance>
 <instance part="CN1" gate="G$1" x="20.32" y="139.7"/>
-<instance part="C" gate="G$1" x="91.44" y="142.24"/>
-<instance part="R" gate="G$1" x="88.9" y="134.62" rot="R180"/>
 <instance part="U$2" gate="G$1" x="33.02" y="127"/>
 <instance part="U$3" gate="G$1" x="76.2" y="129.54"/>
@@
 <instance part="C2" gate="G$1" x="157.48" y="142.24"/>
 <instance part="J1" gate="G$1" x="220.98" y="86.36" rot="R180"/>
+<instance part="D1" gate="G$1" x="88.9" y="142.24" smashed="yes">
+<attribute name="NAME" x="86.106" y="152.908" size="1.016" layer="95" font="vector" align="top-left"/>
+<attribute name="VALUE" x="86.36" y="149.86" size="1.016" layer="96" font="vector"/>
+</instance>
+<instance part="D2" gate="G$1" x="88.9" y="134.62" smashed="yes" rot="R180">
+<attribute name="NAME" x="91.44" y="129.54" size="1.016" layer="95" font="vector" rot="R180" align="top-left"/>
+<attribute name="VALUE" x="104.648" y="128.778" size="1.016" layer="96" font="vector" rot="R180"/>
+</instance>
 </instances>
 <busses>
@@
 <pinref part="U$7" gate="G$1" pin="GND"/>
 <wire x1="83.82" y1="134.62" x2="83.82" y2="132.08" width="0.1524" layer="91"/>
-<pinref part="R" gate="G$1" pin="C"/>
 <wire x1="86.36" y1="134.62" x2="83.82" y2="134.62" width="0.1524" layer="91"/>
+<pinref part="D2" gate="G$1" pin="CATHODE"/>
 </segment>
 <segment>
@@
 <net name="N$1" class="0">
 <segment>
-<pinref part="C" gate="G$1" pin="C"/>
-<wire x1="93.98" y1="142.24" x2="96.52" y2="142.24" width="0.1524" layer="91"/>
 <pinref part="R1" gate="G$1" pin="P$1"/>
+<pinref part="D1" gate="G$1" pin="CATHODE"/>
+<wire x1="91.44" y1="142.24" x2="96.52" y2="142.24" width="0.1524" layer="91"/>
 </segment>
 </net>
@@
 <net name="N$6" class="0">
 <segment>
-<pinref part="R" gate="G$1" pin="A"/>
-<wire x1="96.52" y1="134.62" x2="93.98" y2="134.62" width="0.1524" layer="91"/>
 <pinref part="R2" gate="G$1" pin="P$1"/>
+<pinref part="D2" gate="G$1" pin="ANODE"/>
+<wire x1="91.44" y1="134.62" x2="96.52" y2="134.62" width="0.1524" layer="91"/>
 </segment>
 </net>
@@
 <wire x1="83.82" y1="147.32" x2="111.76" y2="147.32" width="0.1524" layer="91"/>
 <wire x1="76.2" y1="144.78" x2="76.2" y2="147.32" width="0.1524" layer="91"/>
-<pinref part="C" gate="G$1" pin="A"/>
 <wire x1="86.36" y1="142.24" x2="83.82" y2="142.24" width="0.1524" layer="91"/>
 <wire x1="83.82" y1="142.24" x2="83.82" y2="147.32" width="0.1524" layer="91"/>
@@
 <junction x="76.2" y="147.32"/>
 <pinref part="C1" gate="G$1" pin="P$1"/>
-</segment>
-<segment>
+<pinref part="D1" gate="G$1" pin="ANODE"/>
+</segment>
+<segment>

Commit message: cleanup
Parts:
- U2: value (none) -> CP2104; HOUSEPART (none) -> no; MPN (none) -> CP2104; POPULATE (none) -> 1
Changed lines of the file:
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@@
 <part name="U$8" library="microbuilder2" deviceset="VBAT" device=""/>
 <part name="U$9" library="microbuilder2" deviceset="VBUS" device=""/>
-<part name="U2" library="microbuilder2" deviceset="CP2104" device=""/>
+<part name="U2" library="microbuilder2" deviceset="CP2104" device="" value="CP2104">
+<attribute name="HOUSEPART" value="no"/>
+<attribute name="MPN" value="CP2104"/>
+<attribute name="POPULATE" value="1"/>
+</part>
 <part name="U$10" library="microbuilder2" deviceset="3.3V" device=""/>
 <part name="U$11" library="microbuilder" deviceset="GND" device=""/>
@@
 <instance part="U$8" gate="G$1" x="43.18" y="167.64"/>
 <instance part="U$9" gate="G$1" x="60.96" y="154.94"/>
-<instance part="U2" gate="G$1" x="53.34" y="60.96"/>
+<instance part="U2" gate="G$1" x="53.34" y="60.96">
+<attribute name="HOUSEPART" x="53.34" y="60.96" size="1.778" layer="96" display="off"/>
+<attribute name="MPN" x="53.34" y="60.96" size="1.778" layer="96" display="off"/>
+<attribute name="POPULATE" x="53.34" y="60.96" size="1.778" layer="96" display="off"/>
+</instance>
 <instance part="U$10" gate="G$1" x="25.4" y="91.44"/>
 <instance part="U$11" gate="G$1" x="12.7" y="66.04"/>
